Commit message: ajouter 4 robot

File: industry_robot/urdf/warehouse_bot.urdf.xacro (robot description, xacro)
@@ -1,10 +1,11 @@
 <?xml version="1.0"?>
-<robot xmlns:xacro="http://www.ros.org/wiki/xacro" name="warehouse_bot">
-    <xacro:arg name="robot_name" default=""/>
-    <xacro:if value="${'$(arg robot_name)' != ''}">
-        <xacro:property name="topic_prefix" value="/$(arg robot_name)" />
-        <xacro:property name="frame_prefix" value="$(arg robot_name)/" />
+<robot xmlns:xacro="http://www.ros.org/wiki/xacro" name="$(arg robot_core_name)">
+    <xacro:arg name="robot_core_name" default="warehouse_bot"/>
+    <xacro:arg name="namespace" default=""/>
+    <xacro:if value="${'$(arg namespace)' != ''}">
+        <xacro:property name="topic_prefix" value="/$(arg namespace)" />
+        <xacro:property name="frame_prefix" value="$(arg namespace)/" />
     </xacro:if>
-    <xacro:if value="${'$(arg robot_name)' == ''}">
+    <xacro:if value="${'$(arg namespace)' == ''}">
         <xacro:property name="topic_prefix" value="" />
         <xacro:property name="frame_prefix" value="" />
