Commit message: modification du robot

File: industry_robot/urdf/gazebo_control.xacro (robot description, xacro)
@@ -8,9 +8,9 @@
     <!-- ============================================================
          PLUGIN DIFFERENTIAL DRIVE (gz-sim-diff-drive-system)
-         Contrôle les 2 roues motrices arrière via /cmd_vel.
+         Contrôle les 4 roues motrices via /cmd_vel (skid-steer mode).
          Publie l'odométrie sur /odom et la TF odom → base_footprint.
          Paramètres cinématiques :
-           - wheel_separation = 2 × wheel_y_offset = 2 × 0.165 = 0.33 m
-           - wheel_radius = 0.065 m
+           - wheel_separation = 2 × wheel_y_offset = 2 × 0.315 = 0.63 m
+           - wheel_radius = 0.125 m
            - Vitesse max linéaire : ±1.0 m/s
            - Vitesse max angulaire : ±2.0 rad/s
@@ -19,10 +19,13 @@
         <plugin filename="gz-sim-diff-drive-system"
                 name="gz::sim::systems::DiffDrive">
-            <!-- Articulations des roues motrices -->
-            <left_joint>left_wheel_joint</left_joint>
-            <right_joint>right_wheel_joint</right_joint>
+            <!-- Articulations des roues motrices gauches -->
+            <left_joint>front_left_wheel_joint</left_joint>
+            <left_joint>rear_left_wheel_joint</left_joint>
+            <!-- Articulations des roues motrices droites -->
+            <right_joint>front_right_wheel_joint</right_joint>
+            <right_joint>rear_right_wheel_joint</right_joint>
             <!-- Géométrie des roues (cohérent avec robot_core.xacro) -->
-            <wheel_separation>0.33</wheel_separation>
-            <wheel_radius>0.065</wheel_radius>
+            <wheel_separation>0.63</wheel_separation>
+            <wheel_radius>0.125</wheel_radius>
             <!-- Topics de communication -->
             <topic>cmd_vel</topic>
@@ -55,6 +58,8 @@
                 name="gz::sim::systems::JointStatePublisher">
             <topic>joint_states</topic>
-            <joint_name>left_wheel_joint</joint_name>
-            <joint_name>right_wheel_joint</joint_name>
+            <joint_name>front_left_wheel_joint</joint_name>
+            <joint_name>rear_left_wheel_joint</joint_name>
+            <joint_name>front_right_wheel_joint</joint_name>
+            <joint_name>rear_right_wheel_joint</joint_name>
         </plugin>
     </gazebo>

File: industry_robot/urdf/robot_core.xacro (robot description, xacro)
@@ -3,28 +3,24 @@
 <robot xmlns:xacro="http://www.ros.org/wiki/xacro">
     <!-- Châssis principal -->
-    <xacro:property name="chassis_length" value="0.35"/>
-    <xacro:property name="chassis_width"  value="0.30"/>
-    <xacro:property name="chassis_height" value="0.12"/>
-    <xacro:property name="chassis_mass"   value="3.0"/>
-    <!-- Roues motrices (arrière) -->
-    <xacro:property name="wheel_radius"   value="0.065"/>
-    <xacro:property name="wheel_width"    value="0.03"/>
-    <xacro:property name="wheel_mass"     value="0.25"/>
-    <xacro:property name="wheel_x_offset" value="-0.08"/>
-    <xacro:property name="wheel_y_offset" value="0.165"/>
-    <!-- Roue folle (avant) -->
-    <xacro:property name="caster_radius"  value="0.025"/>
-    <xacro:property name="caster_mass"    value="0.1"/>
+    <xacro:property name="chassis_length" value="1.0"/>
+    <xacro:property name="chassis_width"  value="0.55"/>
+    <xacro:property name="chassis_height" value="0.30"/>
+    <xacro:property name="chassis_mass"   value="40.0"/>
+    <!-- Roues (4 roues motrices ou libres, type skid-steer) -->
+    <xacro:property name="wheel_radius"   value="0.125"/>
+    <xacro:property name="wheel_width"    value="0.08"/>
+    <xacro:property name="wheel_mass"     value="3.0"/>
+    <xacro:property name="wheel_x_offset" value="0.35"/>
+    <xacro:property name="wheel_y_offset" value="0.315"/>
     <!-- Plateau cargo -->
-    <xacro:property name="cargo_length"   value="0.30"/>
-    <xacro:property name="cargo_width"    value="0.25"/>
-    <xacro:property name="cargo_height"   value="0.01"/>
-    <xacro:property name="cargo_mass"     value="0.3"/>
-    <xacro:property name="cargo_z_offset" value="0.11"/>
+    <xacro:property name="cargo_length"   value="1.20"/>
+    <xacro:property name="cargo_width"    value="0.70"/>
+    <xacro:property name="cargo_height"   value="0.05"/>
+    <xacro:property name="cargo_mass"     value="5.0"/>
     <!-- Mât avant (support LiDAR + phares) -->
-    <xacro:property name="mast_length"    value="0.04"/>
-    <xacro:property name="mast_width"     value="0.20"/>
-    <xacro:property name="mast_height"    value="0.10"/>
-    <xacro:property name="mast_mass"      value="0.3"/>
+    <xacro:property name="mast_length"    value="0.10"/>
+    <xacro:property name="mast_width"     value="0.35"/>
+    <xacro:property name="mast_height"    value="0.15"/>
+    <xacro:property name="mast_mass"      value="2.0"/>
     <!-- COULEURS (materials URDF pour RViz) -->
     <material name="light_grey">  <color rgba="0.78 0.78 0.78 1.0"/> </material>
@@ -36,4 +32,5 @@
     <material name="orange">      <color rgba="1.0 0.55 0.0 1.0"/>   </material>
     <material name="green_led">   <color rgba="0.2 0.9 0.2 1.0"/>    </material>
+    <material name="blue">        <color rgba="0.1 0.4 0.9 1.0"/>    </material>
     <!-- projection au sol du robot (z = 0) -->
     <link name="base_footprint"/>
@@ -72,91 +69,72 @@
         <material>Gazebo/Grey</material>
     </gazebo>
-    <!-- ROUE GAUCHE (motrice, arrière gauche) Attachée à base_link, orientée pour tourner autour de Y. -->
-    <joint name="left_wheel_joint" type="continuous">
-        <parent link="base_link"/>
-        <child link="left_wheel_link"/>
-        <origin xyz="${wheel_x_offset} ${wheel_y_offset} 0" rpy="-1.5708 0 0"/>
-        <axis xyz="0 0 1"/>
-    </joint>
-    <link name="left_wheel_link">
-        <visual>
-            <geometry>
-                <cylinder radius="${wheel_radius}" length="${wheel_width}"/>
-            </geometry>
-            <material name="black"/>
-        </visual>
-        <collision>
-            <geometry>
-                <cylinder radius="${wheel_radius}" length="${wheel_width}"/>
-            </geometry>
-        </collision>
-        <xacro:inertial_cylinder mass="${wheel_mass}" length="${wheel_width}" radius="${wheel_radius}">
-            <origin xyz="0 0 0" rpy="0 0 0"/>
-        </xacro:inertial_cylinder>
-    </link>
-    <gazebo reference="left_wheel_link">
-        <material>Gazebo/FlatBlack</material>
-        <mu1>0.9</mu1>
-        <mu2>0.9</mu2>
-    </gazebo>
-    <!-- ROUE DROITE (motrice, arrière droite) Symétrique de la roue gauche par rapport au plan xz -->
-    <joint name="right_wheel_joint" type="continuous">
-        <parent link="base_link"/>
-        <child link="right_wheel_link"/>
-        <origin xyz="${wheel_x_offset} -${wheel_y_offset} 0" rpy="1.5708 0 0"/>
-        <axis xyz="0 0 -1"/>
-    </joint>
-    <link name="right_wheel_link">
-        <visual>
-            <geometry>
-                <cylinder radius="${wheel_radius}" length="${wheel_width}"/>
-            </geometry>
-            <material name="black"/>
-        </visual>
-        <collision>
-            <geometry>
-                <cylinder radius="${wheel_radius}" length="${wheel_width}"/>
-            </geometry>
-        </collision>
-        <xacro:inertial_cylinder mass="${wheel_mass}" length="${wheel_width}" radius="${wheel_radius}">
-            <origin xyz="0 0 0" rpy="0 0 0"/>
-        </xacro:inertial_cylinder>
-    </link>
-    <gazebo reference="right_wheel_link">
-        <material>Gazebo/FlatBlack</material>
-        <mu1>0.9</mu1>
-        <mu2>0.9</mu2>
-    </gazebo>
-    <!-- ROUE FOLLE AVANT (caster ball) -->
-    <joint name="caster_wheel_joint" type="fixed">
-        <parent link="chassis_link"/>
-        <child link="caster_wheel_link"/>
-        <origin xyz="0.13 0 -0.10" rpy="0 0 0"/>
-    </joint>
-    <link name="caster_wheel_link">
-        <visual>
-            <geometry>
-                <sphere radius="${caster_radius}"/>
-            </geometry>
-            <material name="dark_grey"/>
-        </visual>
-        <collision>
-            <geometry>
-                <sphere radius="${caster_radius}"/>
-            </geometry>
-        </collision>
-        <xacro:inertial_sphere mass="${caster_mass}" radius="${caster_radius}">
-            <origin xyz="0 0 0" rpy="0 0 0"/>
-        </xacro:inertial_sphere>
-    </link>
-    <gazebo reference="caster_wheel_link">
-        <material>Gazebo/DarkGrey</material>
-        <mu1>0.001</mu1>
-        <mu2>0.001</mu2>
-    </gazebo>
+    <!-- MACROS POUR LES 4 ROUES -->
+    <xacro:macro name="left_wheel" params="prefix x_offset">
+        <joint name="${prefix}_left_wheel_joint" type="continuous">
+            <parent link="base_link"/>
+            <child link="${prefix}_left_wheel_link"/>
+            <origin xyz="${x_offset} ${wheel_y_offset} 0" rpy="-1.5708 0 0"/>
+            <axis xyz="0 0 1"/>
+        </joint>
+        <link name="${prefix}_left_wheel_link">
+            <visual>
+                <geometry>
+                    <cylinder radius="${wheel_radius}" length="${wheel_width}"/>
+                </geometry>
+                <material name="black"/>
+            </visual>
+            <collision>
+                <geometry>
+                    <cylinder radius="${wheel_radius}" length="${wheel_width}"/>
+                </geometry>
+            </collision>
+            <xacro:inertial_cylinder mass="${wheel_mass}" length="${wheel_width}" radius="${wheel_radius}">
+                <origin xyz="0 0 0" rpy="0 0 0"/>
+            </xacro:inertial_cylinder>
+        </link>
+        <gazebo reference="${prefix}_left_wheel_link">
+            <material>Gazebo/FlatBlack</material>
+            <mu1>0.9</mu1>
+            <mu2>0.9</mu2>
+        </gazebo>
+    </xacro:macro>
+    <xacro:macro name="right_wheel" params="prefix x_offset">
+        <joint name="${prefix}_right_wheel_joint" type="continuous">
+            <parent link="base_link"/>
+            <child link="${prefix}_right_wheel_link"/>
+            <origin xyz="${x_offset} -${wheel_y_offset} 0" rpy="1.5708 0 0"/>
+            <axis xyz="0 0 -1"/>
+        </joint>
+        <link name="${prefix}_right_wheel_link">
+            <visual>
+                <geometry>
+                    <cylinder radius="${wheel_radius}" length="${wheel_width}"/>
+                </geometry>
+                <material name="black"/>
+            </visual>
+            <collision>
+                <geometry>
+                    <cylinder radius="${wheel_radius}" length="${wheel_width}"/>
+                </geometry>
+            </collision>
+            <xacro:inertial_cylinder mass="${wheel_mass}" length="${wheel_width}" radius="${wheel_radius}">
+                <origin xyz="0 0 0" rpy="0 0 0"/>
+            </xacro:inertial_cylinder>
+        </link>
+        <gazebo reference="${prefix}_right_wheel_link">
+            <material>Gazebo/FlatBlack</material>
+            <mu1>0.9</mu1>
+            <mu2>0.9</mu2>
+        </gazebo>
+    </xacro:macro>
+    <!-- Instanciation des 4 roues -->
+    <xacro:left_wheel prefix="front" x_offset="${wheel_x_offset}"/>
+    <xacro:left_wheel prefix="rear" x_offset="-${wheel_x_offset}"/>
+    <xacro:right_wheel prefix="front" x_offset="${wheel_x_offset}"/>
+    <xacro:right_wheel prefix="rear" x_offset="-${wheel_x_offset}"/>
     <!-- PILIERS DE SUPPORT — 4 montants reliant le châssis au plateau -->
-    <xacro:property name="post_radius" value="0.008"/>
-    <xacro:property name="post_length" value="0.045"/>
-    <xacro:property name="post_z" value="${chassis_height/2 + post_length/2 + 0.005}"/>
+    <xacro:property name="post_radius" value="0.02"/>
+    <xacro:property name="post_length" value="0.20"/>
+    <xacro:property name="post_z" value="${chassis_height/2 + post_length/2}"/>
     <xacro:macro name="support_post" params="prefix x y">
         <joint name="${prefix}_post_joint" type="fixed">
@@ -172,5 +150,10 @@
                 <material name="dark_grey"/>
             </visual>
-            <xacro:inertial_cylinder mass="0.03" length="${post_length}" radius="${post_radius}">
+            <collision>
+                <geometry>
+                    <cylinder radius="${post_radius}" length="${post_length}"/>
+                </geometry>
+            </collision>
+            <xacro:inertial_cylinder mass="0.2" length="${post_length}" radius="${post_radius}">
                 <origin xyz="0 0 0" rpy="0 0 0"/>
             </xacro:inertial_cylinder>
@@ -181,9 +164,10 @@
     </xacro:macro>
     <!-- Instanciation des 4 piliers aux coins du plateau -->
-    <xacro:support_post prefix="front_left"  x="0.11"  y="0.09"/>
-    <xacro:support_post prefix="front_right" x="0.11"  y="-0.09"/>
-    <xacro:support_post prefix="rear_left"   x="-0.11" y="0.09"/>
-    <xacro:support_post prefix="rear_right"  x="-0.11" y="-0.09"/>
+    <xacro:support_post prefix="front_left"  x="0.4"  y="0.2"/>
+    <xacro:support_post prefix="front_right" x="0.4"  y="-0.2"/>
+    <xacro:support_post prefix="rear_left"   x="-0.4" y="0.2"/>
+    <xacro:support_post prefix="rear_right"  x="-0.4" y="-0.2"/>
     <!--  PLATEAU CARGO — surface plate pour transporter les cartons -->
+    <xacro:property name="cargo_z_offset" value="${chassis_height/2 + post_length + cargo_height/2}"/>
     <joint name="cargo_platform_joint" type="fixed">
         <parent link="chassis_link"/>
@@ -197,5 +181,5 @@
                 <box size="${cargo_length} ${cargo_width} ${cargo_height}"/>
             </geometry>
-            <material name="dark_grey"/>
+            <material name="light_grey"/>
         </visual>
         <collision>
@@ -210,8 +194,8 @@
     </link>
     <gazebo reference="cargo_platform_link">
-        <material>Gazebo/DarkGrey</material>
-    </gazebo>
-    <!-- RAILS LATÉRAUX — garde-corps sur le plateau  -->
-    <xacro:macro name="side_rail" params="prefix y_pos">
+        <material>Gazebo/White</material>
+    </gazebo>
+    <!-- RAILS LATÉRAUX — décoration sur le plateau pour correspondre à l'image -->
+    <xacro:macro name="side_rail" params="prefix y_pos color">
         <joint name="${prefix}_rail_joint" type="fixed">
             <parent link="cargo_platform_link"/>
@@ -222,28 +206,28 @@
             <visual>
                 <geometry>
-                    <box size="${cargo_length} 0.008 0.04"/>
-                </geometry>
-                <material name="light_grey"/>
-            </visual>
-            <xacro:inertial_box mass="0.06" x="${cargo_length}" y="0.008" z="0.04">
+                    <box size="${cargo_length} 0.02 0.05"/>
+                </geometry>
+                <material name="${color}"/>
+            </visual>
+            <xacro:inertial_box mass="0.5" x="${cargo_length}" y="0.02" z="0.05">
                 <origin xyz="0 0 0" rpy="0 0 0"/>
             </xacro:inertial_box>
         </link>
         <gazebo reference="${prefix}_rail_link">
-            <material>Gazebo/Grey</material>
-        </gazebo>
-    </xacro:macro>
-    <xacro:side_rail prefix="left"  y_pos="0.12"/>
-    <xacro:side_rail prefix="right" y_pos="-0.12"/>
+            <material>Gazebo/Blue</material>
+        </gazebo>
+    </xacro:macro>
+    <xacro:side_rail prefix="left"  y_pos="0.34" color="blue"/>
+    <xacro:side_rail prefix="right" y_pos="-0.34" color="blue"/>
     <!-- PARE-CHOCS AVANT — barre de protection industrielle -->
     <joint name="front_bumper_joint" type="fixed">
         <parent link="chassis_link"/>
         <child link="front_bumper_link"/>
-        <origin xyz="${chassis_length/2 + 0.01} 0 -0.03" rpy="0 0 0"/>
+        <origin xyz="${chassis_length/2 + 0.02} 0 -0.10" rpy="0 0 0"/>
     </joint>
     <link name="front_bumper_link">
         <visual>
             <geometry>
-                <box size="0.015 ${chassis_width + 0.02} 0.025"/>
+                <box size="0.04 ${chassis_width + 0.10} 0.05"/>
             </geometry>
             <material name="dark_grey"/>
@@ -251,8 +235,8 @@
         <collision>
             <geometry>
-                <box size="0.015 ${chassis_width + 0.02} 0.025"/>
+                <box size="0.04 ${chassis_width + 0.10} 0.05"/>
             </geometry>
         </collision>
-        <xacro:inertial_box mass="0.1" x="0.015" y="${chassis_width + 0.02}" z="0.025">
+        <xacro:inertial_box mass="1.0" x="0.04" y="${chassis_width + 0.10}" z="0.05">
             <origin xyz="0 0 0" rpy="0 0 0"/>
         </xacro:inertial_box>
@@ -265,5 +249,5 @@
         <parent link="chassis_link"/>
         <child link="front_mast_link"/>
-        <origin xyz="0.13 0 0.12" rpy="0 0 0"/>
+        <origin xyz="${chassis_length/2 - 0.05} 0 ${chassis_height/2 + mast_height/2}" rpy="0 0 0"/>
     </joint>
     <link name="front_mast_link">
@@ -272,5 +256,5 @@
                 <box size="${mast_length} ${mast_width} ${mast_height}"/>
             </geometry>
-            <material name="light_grey"/>
+            <material name="silver"/>
         </visual>
         <collision>
@@ -290,10 +274,10 @@
         <parent link="front_mast_link"/>
         <child link="estop_link"/>
-        <origin xyz="0.025 -0.08 0.03" rpy="0 1.5708 0"/>
+        <origin xyz="0.05 -0.12 0.05" rpy="0 1.5708 0"/>
     </joint>
     <link name="estop_link">
         <visual>
             <geometry>
-                <cylinder radius="0.015" length="0.015"/>
+                <cylinder radius="0.02" length="0.02"/>
             </geometry>
             <material name="red"/>
@@ -303,15 +287,15 @@
         <material>Gazebo/Red</material>
     </gazebo>
-    <!--  PHARES AVANT — 2 petites lumières LED sur le mât -->
+    <!--  PHARES AVANT — 2 lumières LED sur le mât -->
     <xacro:macro name="headlight" params="prefix y_offset">
         <joint name="${prefix}_light_joint" type="fixed">
             <parent link="front_mast_link"/>
             <child link="${prefix}_light_link"/>
-            <origin xyz="0.025 ${y_offset} -0.02" rpy="0 1.5708 0"/>
+            <origin xyz="0.051 ${y_offset} -0.04" rpy="0 1.5708 0"/>
         </joint>
         <link name="${prefix}_light_link">
             <visual>
                 <geometry>
-                    <cylinder radius="0.01" length="0.008"/>
+                    <cylinder radius="0.02" length="0.01"/>
                 </geometry>
                 <material name="yellow"/>
@@ -322,16 +306,16 @@
         </gazebo>
     </xacro:macro>
-    <xacro:headlight prefix="left_head"  y_offset="0.04"/>
-    <xacro:headlight prefix="right_head" y_offset="-0.04"/>
+    <xacro:headlight prefix="left_head"  y_offset="0.10"/>
+    <xacro:headlight prefix="right_head" y_offset="-0.10"/>
     <!-- INDICATEUR LED STATUS — petit voyant vert sur le mât -->
     <joint name="status_led_joint" type="fixed">
         <parent link="front_mast_link"/>
         <child link="status_led_link"/>
-        <origin xyz="0.025 0 0.04" rpy="0 1.5708 0"/>
+        <origin xyz="0.051 0 0.05" rpy="0 1.5708 0"/>
     </joint>
     <link name="status_led_link">
         <visual>
             <geometry>
-                <cylinder radius="0.006" length="0.005"/>
+                <cylinder radius="0.01" length="0.01"/>
             </geometry>
             <material name="green_led"/>

Commit message: add plusieur robot

File: industry_robot/urdf/gazebo_control.xacro (robot description, xacro)
@@ -29,10 +29,10 @@
             <wheel_radius>0.125</wheel_radius>
             <!-- Topics de communication -->
-            <topic>cmd_vel</topic>
-            <odom_topic>odom</odom_topic>
-            <tf_topic>/tf</tf_topic>
+            <topic>${topic_prefix}/cmd_vel</topic>
+            <odom_topic>${topic_prefix}/odom</odom_topic>
+            <tf_topic>${topic_prefix}/tf</tf_topic>
             <!-- Frames de l'odométrie -->
-            <frame_id>odom</frame_id>
-            <child_frame_id>base_footprint</child_frame_id>
+            <frame_id>${frame_prefix}odom</frame_id>
+            <child_frame_id>${frame_prefix}base_footprint</child_frame_id>
             <!-- Fréquence de publication de l'odométrie (Hz) -->
             <odom_publish_frequency>50</odom_publish_frequency>
@@ -57,5 +57,5 @@
         <plugin filename="gz-sim-joint-state-publisher-system"
                 name="gz::sim::systems::JointStatePublisher">
-            <topic>joint_states</topic>
+            <topic>${topic_prefix}/joint_states</topic>
             <joint_name>front_left_wheel_joint</joint_name>
             <joint_name>rear_left_wheel_joint</joint_name>

File: industry_robot/urdf/imu.xacro (robot description, xacro)
@@ -37,7 +37,7 @@
         <sensor name="imu_sensor" type="imu">
             <pose>0 0 0 0 0 0</pose>
-            <topic>imu</topic>
+            <topic>${topic_prefix}/imu</topic>
             <update_rate>50</update_rate>
-            <gz_frame_id>imu_link</gz_frame_id>
+            <gz_frame_id>${frame_prefix}imu_link</gz_frame_id>
             <always_on>1</always_on>
             <visualize>false</visualize>

File: industry_robot/urdf/lidar.xacro (robot description, xacro)
@@ -40,7 +40,7 @@
         <sensor name="lidar" type="gpu_lidar">
             <pose>0 0 0 0 0 0</pose>
-            <topic>scan</topic>
+            <topic>${topic_prefix}/scan</topic>
             <update_rate>10</update_rate>
-            <gz_frame_id>lidar_link</gz_frame_id>
+            <gz_frame_id>${frame_prefix}lidar_link</gz_frame_id>
             <lidar>
                 <scan>

File: industry_robot/urdf/warehouse_bot.urdf.xacro (robot description, xacro)
@@ -1,4 +1,13 @@
 <?xml version="1.0"?>
 <robot xmlns:xacro="http://www.ros.org/wiki/xacro" name="warehouse_bot">
+    <xacro:arg name="robot_name" default=""/>
+    <xacro:if value="${'$(arg robot_name)' != ''}">
+        <xacro:property name="topic_prefix" value="/$(arg robot_name)" />
+        <xacro:property name="frame_prefix" value="$(arg robot_name)/" />
+    </xacro:if>
+    <xacro:if value="${'$(arg robot_name)' == ''}">
+        <xacro:property name="topic_prefix" value="" />
+        <xacro:property name="frame_prefix" value="" />
+    </xacro:if>
     <!-- Inclure les macros d'inertie -->
     <xacro:include filename="inertial_macros.xacro"/>
