Commit message: deplacement des robot

File: industry_robot/urdf/gazebo_control.xacro (robot description, xacro)
@@ -28,8 +28,5 @@
             <wheel_separation>0.63</wheel_separation>
             <wheel_radius>0.125</wheel_radius>
-            <!-- Topics de communication -->
-            <topic>${topic_prefix}/cmd_vel</topic>
-            <odom_topic>${topic_prefix}/odom</odom_topic>
-            <tf_topic>${topic_prefix}/tf</tf_topic>
+            <!-- Topics de communication supprimés pour utiliser les valeurs par défaut de Gazebo (/model/robot1/cmd_vel) -->
             <!-- Frames de l'odométrie -->
             <frame_id>${frame_prefix}odom</frame_id>
@@ -57,5 +54,5 @@
         <plugin filename="gz-sim-joint-state-publisher-system"
                 name="gz::sim::systems::JointStatePublisher">
-            <topic>${topic_prefix}/joint_states</topic>
+            <topic>joint_states</topic>
             <joint_name>front_left_wheel_joint</joint_name>
             <joint_name>rear_left_wheel_joint</joint_name>

File: industry_robot/urdf/robot_core.xacro (robot description, xacro)
@@ -86,5 +86,5 @@
             <collision>
                 <geometry>
-                    <cylinder radius="${wheel_radius}" length="${wheel_width}"/>
+                    <sphere radius="${wheel_radius}"/>
                 </geometry>
             </collision>
@@ -115,5 +115,5 @@
             <collision>
                 <geometry>
-                    <cylinder radius="${wheel_radius}" length="${wheel_width}"/>
+                    <sphere radius="${wheel_radius}"/>
                 </geometry>
             </collision>

Commit message: activation du lidar

File: industry_robot/urdf/gazebo_control.xacro (robot description, xacro)
@@ -37,4 +37,8 @@
             <frame_id>${frame_prefix}odom</frame_id>
             <child_frame_id>${frame_prefix}base_footprint</child_frame_id>
+            <odometry_frame>${frame_prefix}odom</odometry_frame>
+            <robot_base_frame>${frame_prefix}base_footprint</robot_base_frame>
+            <publish_odom>true</publish_odom>
+            <publish_odom_tf>true</publish_odom_tf>
             <!-- Fréquence de publication de l'odométrie (Hz) -->
             <odom_publish_frequency>50</odom_publish_frequency>

File: industry_robot/urdf/lidar.xacro (robot description, xacro)
@@ -37,5 +37,5 @@
     -->
     <gazebo reference="lidar_link">
-        <material>Gazebo/FlatBlack</material>
+        <material>Gazebo/Red</material>
         <sensor name="lidar" type="gpu_lidar">
             <pose>0 0 0 0 0 0</pose>
