Commit message: ACTIVATION DU LIDAR

File: industry_robot/urdf/imu.xacro (robot description, xacro)
@@ -27,5 +27,5 @@
         <sensor name="imu_sensor" type="imu">
             <pose>0 0 0 0 0 0</pose>
-            <topic>${topic_prefix}/imu</topic>
+            <topic>imu</topic>
             <update_rate>50</update_rate>
             <gz_frame_id>${frame_prefix}imu_link</gz_frame_id>

File: industry_robot/urdf/lidar.xacro (robot description, xacro)
@@ -9,5 +9,5 @@
         <parent link="front_mast_link"/>
         <child link="lidar_link"/>
-        <origin xyz="0 0 0.07" rpy="0 0 0"/>
+        <origin xyz="0 0 0.25" rpy="0 0 0"/>
     </joint>
     <link name="lidar_link">
@@ -40,5 +40,5 @@
         <sensor name="lidar" type="gpu_lidar">
             <pose>0 0 0 0 0 0</pose>
-            <topic>${topic_prefix}/scan</topic>
+            <topic>scan</topic>
             <update_rate>10</update_rate>
             <gz_frame_id>${frame_prefix}lidar_link</gz_frame_id>

File: industry_robot/urdf/robot_core.xacro (robot description, xacro)
@@ -21,5 +21,5 @@
     <xacro:property name="mast_length"    value="0.10"/>
     <xacro:property name="mast_width"     value="0.35"/>
-    <xacro:property name="mast_height"    value="0.15"/>
+    <xacro:property name="mast_height"    value="0.45"/>
     <xacro:property name="mast_mass"      value="2.0"/>
     <!-- COULEURS (materials URDF pour RViz) -->
