Commit message: adjust height lidar

File: industry_robot/urdf/lidar.xacro (robot description, xacro)
@@ -9,5 +9,5 @@
         <parent link="front_mast_link"/>
         <child link="lidar_link"/>
-        <origin xyz="0 0 0.25" rpy="0 0 0"/>
+        <origin xyz="0 0 0.07" rpy="0 0 0"/>
     </joint>
     <link name="lidar_link">

File: industry_robot/urdf/robot_core.xacro (robot description, xacro)
@@ -21,5 +21,5 @@
     <xacro:property name="mast_length"    value="0.10"/>
     <xacro:property name="mast_width"     value="0.35"/>
-    <xacro:property name="mast_height"    value="0.45"/>
+    <xacro:property name="mast_height"    value="0.15"/>
     <xacro:property name="mast_mass"      value="2.0"/>
     <!-- COULEURS (materials URDF pour RViz) -->
