Commit message: laser filter robot

File: industry_robot/urdf/robot_core.xacro (robot description, xacro)
@@ -177,4 +177,7 @@
         <origin xyz="0 0 ${cargo_z_offset}" rpy="0 0 0"/>
     </joint>
+    <!-- NB: <collision> retiré du plateau cargo pour éviter la self-detection LiDAR.
+         Le plateau reste visible (visual) et conserve sa masse (inertial),
+         mais devient transparent au raycasting du gpu_lidar. -->
     <link name="cargo_platform_link">
         <visual>
@@ -185,10 +188,4 @@
             <material name="light_grey"/>
         </visual>
-        <collision>
-            <origin xyz="0 0 0" rpy="0 0 0"/>
-            <geometry>
-                <box size="${cargo_length} ${cargo_width} ${cargo_height}"/>
-            </geometry>
-        </collision>
         <xacro:inertial_box mass="${cargo_mass}" x="${cargo_length}" y="${cargo_width}" z="${cargo_height}">
             <origin xyz="0 0 0" rpy="0 0 0"/>
