Commit message: modification de urdf

File: industry_robot_description/urdf/gazebo_control.xacro (robot description, xacro)
@@ -25,7 +25,8 @@
             <right_joint>front_right_wheel_joint</right_joint>
             <right_joint>rear_right_wheel_joint</right_joint>
-            <!-- Géométrie des roues (cohérent avec robot_core.xacro) -->
-            <wheel_separation>0.63</wheel_separation>
-            <wheel_radius>0.125</wheel_radius>
+            <!-- Géométrie des roues (cohérent avec nouveau robot_core.xacro style Husky A300) -->
+            <!-- wheel_separation = 2 × wheel_y_offset = 2 × 0.37 = 0.74 m -->
+            <wheel_separation>0.74</wheel_separation>
+            <wheel_radius>0.165</wheel_radius>
             <!-- Topics : laissés en défaut Gazebo Harmonic.
                  GZ crée automatiquement :

File: industry_robot_description/urdf/imu.xacro (robot description, xacro)
@@ -27,5 +27,5 @@
         <sensor name="imu_sensor" type="imu">
             <pose>0 0 0 0 0 0</pose>
-            <topic>imu</topic>
+            <topic>${topic_prefix}/imu</topic>
             <update_rate>50</update_rate>
             <gz_frame_id>${frame_prefix}imu_link</gz_frame_id>

File: industry_robot_description/urdf/lidar.xacro (robot description, xacro)
@@ -7,7 +7,7 @@
     <!--  LIEN ET JOINT DU LiDAR -->
     <joint name="lidar_joint" type="fixed">
-        <parent link="front_mast_link"/>
+        <parent link="sensor_mast_link"/>
         <child link="lidar_link"/>
-        <origin xyz="0 0 0.07" rpy="0 0 0"/>
+        <origin xyz="0 0 0.12" rpy="0 0 0"/>
     </joint>
     <link name="lidar_link">
@@ -40,5 +40,5 @@
         <sensor name="lidar" type="gpu_lidar">
             <pose>0 0 0 0 0 0</pose>
-            <topic>scan</topic>
+            <topic>${topic_prefix}/scan</topic>
             <update_rate>10</update_rate>
             <gz_frame_id>${frame_prefix}lidar_link</gz_frame_id>

File: industry_robot_description/urdf/robot_core.xacro (robot description, xacro)
@@ -2,25 +2,29 @@
 <!-- robot_core.xacro — Corps principal du robot AMR d'entrepôt -->
 <robot xmlns:xacro="http://www.ros.org/wiki/xacro">
-    <!-- Châssis principal -->
-    <xacro:property name="chassis_length" value="1.0"/>
-    <xacro:property name="chassis_width"  value="0.55"/>
-    <xacro:property name="chassis_height" value="0.30"/>
-    <xacro:property name="chassis_mass"   value="40.0"/>
-    <!-- Roues (4 roues motrices ou libres, type skid-steer) -->
-    <xacro:property name="wheel_radius"   value="0.125"/>
-    <xacro:property name="wheel_width"    value="0.08"/>
-    <xacro:property name="wheel_mass"     value="3.0"/>
-    <xacro:property name="wheel_x_offset" value="0.35"/>
-    <xacro:property name="wheel_y_offset" value="0.315"/>
-    <!-- Plateau cargo -->
-    <xacro:property name="cargo_length"   value="1.20"/>
-    <xacro:property name="cargo_width"    value="0.70"/>
-    <xacro:property name="cargo_height"   value="0.05"/>
-    <xacro:property name="cargo_mass"     value="5.0"/>
-    <!-- Mât avant (support LiDAR + phares) -->
+    <!-- Châssis principal (Style Husky A300) -->
+    <xacro:property name="chassis_length" value="0.90"/>
+    <xacro:property name="chassis_width"  value="0.54"/>
+    <xacro:property name="chassis_height" value="0.25"/>
+    <xacro:property name="chassis_mass"   value="45.0"/>
+    <xacro:property name="bumper_length" value="0.08"/>
+    <xacro:property name="bumper_width"  value="0.62"/>
+    <xacro:property name="bumper_height" value="0.11"/>
+    <xacro:property name="bumper_mass"   value="2.0"/>
+    <!-- Roues (4 roues type tout-terrain Husky) -->
+    <xacro:property name="wheel_radius"   value="0.165"/>
+    <xacro:property name="wheel_width"    value="0.114"/>
+    <xacro:property name="wheel_mass"     value="4.0"/>
+    <xacro:property name="wheel_x_offset" value="0.28"/>
+    <xacro:property name="wheel_y_offset" value="0.37"/>
+    <!-- Plateau supérieur (Top Plate) -->
+    <xacro:property name="cargo_length"   value="0.82"/>
+    <xacro:property name="cargo_width"    value="0.48"/>
+    <xacro:property name="cargo_height"   value="0.04"/>
+    <xacro:property name="cargo_mass"     value="3.0"/>
+    <!-- Mât capteurs (LiDAR & IMU) -->
     <xacro:property name="mast_length"    value="0.10"/>
-    <xacro:property name="mast_width"     value="0.35"/>
-    <xacro:property name="mast_height"    value="0.15"/>
-    <xacro:property name="mast_mass"      value="2.0"/>
+    <xacro:property name="mast_width"     value="0.10"/>
+    <xacro:property name="mast_height"    value="0.20"/>
+    <xacro:property name="mast_mass"      value="1.5"/>
     <!-- COULEURS (materials URDF pour RViz) -->
     <material name="light_grey">  <color rgba="0.78 0.78 0.78 1.0"/> </material>
@@ -54,5 +58,5 @@
                 <box size="${chassis_length} ${chassis_width} ${chassis_height}"/>
             </geometry>
-            <material name="silver"/>
+            <material name="dark_grey"/>
         </visual>
         <collision>
@@ -67,6 +71,34 @@
     </link>
     <gazebo reference="chassis_link">
-        <material>Gazebo/Grey</material>
+        <material>Gazebo/DarkGrey</material>
     </gazebo>
+    <xacro:macro name="bumper" params="name x_offset">
+        <joint name="${name}_bumper_joint" type="fixed">
+            <parent link="chassis_link"/>
+            <child link="${name}_bumper_link"/>
+            <origin xyz="${x_offset} 0 -0.02" rpy="0 0 0"/>
+        </joint>
+        <link name="${name}_bumper_link">
+            <visual>
+                <geometry>
+                    <box size="${bumper_length} ${bumper_width} ${bumper_height}"/>
+                </geometry>
+                <material name="black"/>
+            </visual>
+            <collision>
+                <geometry>
+                    <box size="${bumper_length} ${bumper_width} ${bumper_height}"/>
+                </geometry>
+            </collision>
+            <xacro:inertial_box mass="${bumper_mass}" x="${bumper_length}" y="${bumper_width}" z="${bumper_height}">
+                <origin xyz="0 0 0" rpy="0 0 0"/>
+            </xacro:inertial_box>
+        </link>
+        <gazebo reference="${name}_bumper_link">
+            <material>Gazebo/FlatBlack</material>
+        </gazebo>
+    </xacro:macro>
+    <xacro:bumper name="front" x_offset="${chassis_length/2 + bumper_length/2}"/>
+    <xacro:bumper name="rear" x_offset="-${chassis_length/2 + bumper_length/2}"/>
     <!-- MACROS POUR LES 4 ROUES -->
     <xacro:macro name="left_wheel" params="prefix x_offset">
@@ -135,41 +167,6 @@
     <xacro:right_wheel prefix="front" x_offset="${wheel_x_offset}"/>
     <xacro:right_wheel prefix="rear" x_offset="-${wheel_x_offset}"/>
-    <!-- PILIERS DE SUPPORT — 4 montants reliant le châssis au plateau -->
-    <xacro:property name="post_radius" value="0.02"/>
-    <xacro:property name="post_length" value="0.20"/>
-    <xacro:property name="post_z" value="${chassis_height/2 + post_length/2}"/>
-    <xacro:macro name="support_post" params="prefix x y">
-        <joint name="${prefix}_post_joint" type="fixed">
-            <parent link="chassis_link"/>
-            <child link="${prefix}_post_link"/>
-            <origin xyz="${x} ${y} ${post_z}" rpy="0 0 0"/>
-        </joint>
-        <link name="${prefix}_post_link">
-            <visual>
-                <geometry>
-                    <cylinder radius="${post_radius}" length="${post_length}"/>
-                </geometry>
-                <material name="dark_grey"/>
-            </visual>
-            <collision>
-                <geometry>
-                    <cylinder radius="${post_radius}" length="${post_length}"/>
-                </geometry>
-            </collision>
-            <xacro:inertial_cylinder mass="0.2" length="${post_length}" radius="${post_radius}">
-                <origin xyz="0 0 0" rpy="0 0 0"/>
-            </xacro:inertial_cylinder>
-        </link>
-        <gazebo reference="${prefix}_post_link">
-            <material>Gazebo/DarkGrey</material>
-        </gazebo>
-    </xacro:macro>
-    <!-- Instanciation des 4 piliers aux coins du plateau -->
-    <xacro:support_post prefix="front_left"  x="0.4"  y="0.2"/>
-    <xacro:support_post prefix="front_right" x="0.4"  y="-0.2"/>
-    <xacro:support_post prefix="rear_left"   x="-0.4" y="0.2"/>
-    <xacro:support_post prefix="rear_right"  x="-0.4" y="-0.2"/>
-    <!--  PLATEAU CARGO — surface plate pour transporter les cartons -->
-    <xacro:property name="cargo_z_offset" value="${chassis_height/2 + post_length + cargo_height/2}"/>
+    <!--  PLATEAU SUPÉRIEUR — top plate du Husky -->
+    <xacro:property name="cargo_z_offset" value="${chassis_height/2 + cargo_height/2}"/>
     <joint name="cargo_platform_joint" type="fixed">
         <parent link="chassis_link"/>
@@ -186,5 +183,5 @@
                 <box size="${cargo_length} ${cargo_width} ${cargo_height}"/>
             </geometry>
-            <material name="light_grey"/>
+            <material name="dark_grey"/>
         </visual>
         <xacro:inertial_box mass="${cargo_mass}" x="${cargo_length}" y="${cargo_width}" z="${cargo_height}">
@@ -193,65 +190,16 @@
     </link>
     <gazebo reference="cargo_platform_link">
-        <material>Gazebo/White</material>
-    </gazebo>
-    <!-- RAILS LATÉRAUX — décoration sur le plateau pour correspondre à l'image -->
-    <xacro:macro name="side_rail" params="prefix y_pos color">
-        <joint name="${prefix}_rail_joint" type="fixed">
-            <parent link="cargo_platform_link"/>
-            <child link="${prefix}_rail_link"/>
-            <origin xyz="0 ${y_pos} 0.025" rpy="0 0 0"/>
-        </joint>
-        <link name="${prefix}_rail_link">
-            <visual>
-                <geometry>
-                    <box size="${cargo_length} 0.02 0.05"/>
-                </geometry>
-                <material name="${color}"/>
-            </visual>
-            <xacro:inertial_box mass="0.5" x="${cargo_length}" y="0.02" z="0.05">
-                <origin xyz="0 0 0" rpy="0 0 0"/>
-            </xacro:inertial_box>
-        </link>
-        <gazebo reference="${prefix}_rail_link">
-            <material>Gazebo/Blue</material>
-        </gazebo>
-    </xacro:macro>
-    <xacro:side_rail prefix="left"  y_pos="0.34" color="blue"/>
-    <xacro:side_rail prefix="right" y_pos="-0.34" color="blue"/>
-    <!-- PARE-CHOCS AVANT — barre de protection industrielle -->
-    <joint name="front_bumper_joint" type="fixed">
-        <parent link="chassis_link"/>
-        <child link="front_bumper_link"/>
-        <origin xyz="${chassis_length/2 + 0.02} 0 -0.10" rpy="0 0 0"/>
-    </joint>
-    <link name="front_bumper_link">
-        <visual>
-            <geometry>
-                <box size="0.04 ${chassis_width + 0.10} 0.05"/>
-            </geometry>
-            <material name="dark_grey"/>
-        </visual>
-        <collision>
-            <geometry>
-                <box size="0.04 ${chassis_width + 0.10} 0.05"/>
-            </geometry>
-        </collision>
-        <xacro:inertial_box mass="1.0" x="0.04" y="${chassis_width + 0.10}" z="0.05">
-            <origin xyz="0 0 0" rpy="0 0 0"/>
-        </xacro:inertial_box>
-    </link>
-    <gazebo reference="front_bumper_link">
         <material>Gazebo/DarkGrey</material>
     </gazebo>
-    <!--  MÂT AVANT — structure portant le LiDAR et les phares  -->
-    <joint name="front_mast_joint" type="fixed">
-        <parent link="chassis_link"/>
-        <child link="front_mast_link"/>
-        <origin xyz="${chassis_length/2 - 0.05} 0 ${chassis_height/2 + mast_height/2}" rpy="0 0 0"/>
-    </joint>
-    <link name="front_mast_link">
+    <!--  MÂT CAPTEURS — structure centrale pour LiDAR et IMU  -->
+    <joint name="sensor_mast_joint" type="fixed">
+        <parent link="cargo_platform_link"/>
+        <child link="sensor_mast_link"/>
+        <origin xyz="0.25 0 ${cargo_height/2 + mast_height/2}" rpy="0 0 0"/>
+    </joint>
+    <link name="sensor_mast_link">
         <visual>
             <geometry>
-                <box size="${mast_length} ${mast_width} ${mast_height}"/>
+                <cylinder radius="${mast_width/2}" length="${mast_height}"/>
             </geometry>
             <material name="silver"/>
@@ -259,68 +207,13 @@
         <collision>
             <geometry>
-                <box size="${mast_length} ${mast_width} ${mast_height}"/>
+                <cylinder radius="${mast_width/2}" length="${mast_height}"/>
             </geometry>
         </collision>
-        <xacro:inertial_box mass="${mast_mass}" x="${mast_length}" y="${mast_width}" z="${mast_height}">
-            <origin xyz="0 0 0" rpy="0 0 0"/>
-        </xacro:inertial_box>
+        <xacro:inertial_cylinder mass="${mast_mass}" radius="${mast_width/2}" length="${mast_height}">
+            <origin xyz="0 0 0" rpy="0 0 0"/>
+        </xacro:inertial_cylinder>
     </link>
-    <gazebo reference="front_mast_link">
+    <gazebo reference="sensor_mast_link">
         <material>Gazebo/Grey</material>
     </gazebo>
-    <!--  BOUTON D'ARRÊT D'URGENCE (E-Stop) — visuel décoratif-->
-    <joint name="estop_joint" type="fixed">
-        <parent link="front_mast_link"/>
-        <child link="estop_link"/>
-        <origin xyz="0.05 -0.12 0.05" rpy="0 1.5708 0"/>
-    </joint>
-    <link name="estop_link">
-        <visual>
-            <geometry>
-                <cylinder radius="0.02" length="0.02"/>
-            </geometry>
-            <material name="red"/>
-        </visual>
-    </link>
-    <gazebo reference="estop_link">
-        <material>Gazebo/Red</material>
-    </gazebo>
-    <!--  PHARES AVANT — 2 lumières LED sur le mât -->
-    <xacro:macro name="headlight" params="prefix y_offset">
-        <joint name="${prefix}_light_joint" type="fixed">
-            <parent link="front_mast_link"/>
-            <child link="${prefix}_light_link"/>
-            <origin xyz="0.051 ${y_offset} -0.04" rpy="0 1.5708 0"/>
-        </joint>
-        <link name="${prefix}_light_link">
-            <visual>
-                <geometry>
-                    <cylinder radius="0.02" length="0.01"/>
-                </geometry>
-                <material name="yellow"/>
-            </visual>
-        </link>
-        <gazebo reference="${prefix}_light_link">
-            <material>Gazebo/Yellow</material>
-        </gazebo>
-    </xacro:macro>
-    <xacro:headlight prefix="left_head"  y_offset="0.10"/>
-    <xacro:headlight prefix="right_head" y_offset="-0.10"/>
-    <!-- INDICATEUR LED STATUS — petit voyant vert sur le mât -->
-    <joint name="status_led_joint" type="fixed">
-        <parent link="front_mast_link"/>
-        <child link="status_led_link"/>
-        <origin xyz="0.051 0 0.05" rpy="0 1.5708 0"/>
-    </joint>
-    <link name="status_led_link">
-        <visual>
-            <geometry>
-                <cylinder radius="0.01" length="0.01"/>
-            </geometry>
-            <material name="green_led"/>
-        </visual>
-    </link>
-    <gazebo reference="status_led_link">
-        <material>Gazebo/Green</material>
-    </gazebo>
 </robot>
