Commit message: KAN-13 fix navigation essaie collision

File: industry_robot_description/urdf/imu.xacro (robot description, xacro)
@@ -11,5 +11,7 @@
                 <box size="0.03 0.03 0.01"/>
             </geometry>
-            <material name="yellow"/>
+            <material name="yellow">
+                <color rgba="1.0 1.0 0.0 1.0"/>
+            </material>
         </visual>
         <xacro:inertial_box mass="0.02" x="0.03" y="0.03" z="0.01">
